File: Stecchino_PCB_2/Projet_Stecchino.kicad_pcb (KiCad board)
At the start: 2 copper layers, 97.2 x 31.8 mm, 14 parts, among them P1 CONN_01X02, P2 CONN_01X03, SW1 SW_PUSH, SW2 SW_PUSH

Commit message: Minor changes to PCB to increase hole diameters for mpu and lipo management board
Other:
- board text added: "2.0"
- board text added: "Nov 2018"
- board text removed: "1.0"
- board text removed: "Sept 2017"
Changed lines of the file:
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@@
     (mod_text_size 1 1)
     (mod_text_width 0.15)
-    (pad_size 1.524 1.524)
-    (pad_drill 0.762)
+    (pad_size 2.032 2.032)
+    (pad_drill 1.016)
     (pad_to_mask_clearance 0.2)
     (aux_axis_origin 0 0)
@@
     (fp_line (start -17.145 20.955) (end -17.145 22.86) (layer F.SilkS) (width 0.15))
     (fp_line (start -17.145 22.86) (end -11.43 22.86) (layer F.SilkS) (width 0.15))
-    (pad 1 thru_hole circle (at 7.62 10.16 90) (size 1.524 1.524) (drill 0.762) (layers *.Cu *.Mask F.SilkS)
+    (pad 1 thru_hole circle (at 7.62 10.16 90) (size 2.032 2.032) (drill 1.016) (layers *.Cu *.Mask F.SilkS)
       (net 2 /LIPO+))
-    (pad 2 thru_hole circle (at 7.62 17.78 90) (size 1.524 1.524) (drill 0.762) (layers *.Cu *.Mask F.SilkS)
+    (pad 2 thru_hole circle (at 7.62 17.78 90) (size 2.032 2.032) (drill 1.016) (layers *.Cu *.Mask F.SilkS)
       (net 1 /LIPO-))
-    (pad 4 thru_hole circle (at 7.62 6.985 90) (size 1.524 1.524) (drill 0.762) (layers *.Cu *.Mask F.SilkS)
+    (pad 4 thru_hole circle (at 7.62 6.985 90) (size 2.032 2.032) (drill 1.016) (layers *.Cu *.Mask F.SilkS)
       (net 8 +BATT))
-    (pad 3 thru_hole circle (at 7.62 20.955 90) (size 1.524 1.524) (drill 0.762) (layers *.Cu *.Mask F.SilkS)
+    (pad 3 thru_hole circle (at 7.62 20.955 90) (size 2.032 2.032) (drill 1.016) (layers *.Cu *.Mask F.SilkS)
       (net 5 GND))
-    (pad 5 thru_hole circle (at -15.24 20.955 90) (size 1.524 1.524) (drill 0.762) (layers *.Cu *.Mask F.SilkS)
+    (pad 5 thru_hole circle (at -15.24 20.955 90) (size 2.032 2.032) (drill 1.016) (layers *.Cu *.Mask F.SilkS)
       (net 12 "Net-(U1-Pad5)"))
-    (pad 6 thru_hole circle (at -15.24 6.985 90) (size 1.524 1.524) (drill 0.762) (layers *.Cu *.Mask F.SilkS)
+    (pad 6 thru_hole circle (at -15.24 6.985 90) (size 2.032 2.032) (drill 1.016) (layers *.Cu *.Mask F.SilkS)
       (net 13 "Net-(U1-Pad6)"))
   )
@@
     (fp_line (start 10.16 -2.54) (end -10.16 -2.54) (layer F.SilkS) (width 0.15))
     (fp_line (start -10.16 -2.54) (end -10.16 12.7) (layer F.SilkS) (width 0.15))
-    (pad 1 thru_hole circle (at -8.89 11.43 180) (size 1.524 1.524) (drill 0.762) (layers *.Cu *.Mask F.SilkS)
+    (pad 1 thru_hole circle (at -8.89 11.43 180) (size 2.032 2.032) (drill 1.016) (layers *.Cu *.Mask F.SilkS)
       (net 14 /ITG/MPU_VCC))
-    (pad 2 thru_hole circle (at -6.35 11.43 180) (size 1.524 1.524) (drill 0.762) (layers *.Cu *.Mask F.SilkS)
+    (pad 2 thru_hole circle (at -6.35 11.43 180) (size 2.032 2.032) (drill 1.016) (layers *.Cu *.Mask F.SilkS)
       (net 5 GND))
-    (pad 3 thru_hole circle (at -3.81 11.43 180) (size 1.524 1.524) (drill 0.762) (layers *.Cu *.Mask F.SilkS)
+    (pad 3 thru_hole circle (at -3.81 11.43 180) (size 2.032 2.032) (drill 1.016) (layers *.Cu *.Mask F.SilkS)
       (net 15 /I2C_SCL))
-    (pad 4 thru_hole circle (at -1.27 11.43 180) (size 1.524 1.524) (drill 0.762) (layers *.Cu *.Mask F.SilkS)
+    (pad 4 thru_hole circle (at -1.27 11.43 180) (size 2.032 2.032) (drill 1.016) (layers *.Cu *.Mask F.SilkS)
       (net 16 /I2C_SDA))
-    (pad 5 thru_hole circle (at 1.27 11.43 180) (size 1.524 1.524) (drill 0.762) (layers *.Cu *.Mask F.SilkS)
+    (pad 5 thru_hole circle (at 1.27 11.43 180) (size 2.032 2.032) (drill 1.016) (layers *.Cu *.Mask F.SilkS)
       (net 17 "Net-(U2-Pad5)"))
-    (pad 6 thru_hole circle (at 3.81 11.43 180) (size 1.524 1.524) (drill 0.762) (layers *.Cu *.Mask F.SilkS)
+    (pad 6 thru_hole circle (at 3.81 11.43 180) (size 2.032 2.032) (drill 1.016) (layers *.Cu *.Mask F.SilkS)
       (net 18 "Net-(U2-Pad6)"))
-    (pad 7 thru_hole circle (at 6.35 11.43 180) (size 1.524 1.524) (drill 0.762) (layers *.Cu *.Mask F.SilkS)
+    (pad 7 thru_hole circle (at 6.35 11.43 180) (size 2.032 2.032) (drill 1.016) (layers *.Cu *.Mask F.SilkS)
       (net 19 "Net-(U2-Pad7)"))
-    (pad 8 thru_hole circle (at 8.89 11.43 180) (size 1.524 1.524) (drill 0.762) (layers *.Cu *.Mask F.SilkS)
+    (pad 8 thru_hole circle (at 8.89 11.43 180) (size 2.032 2.032) (drill 1.016) (layers *.Cu *.Mask F.SilkS)
       (net 11 /D3))
   )
@@
   (gr_line (start 93.98 135.255) (end 191.135 135.255) (angle 90) (layer Edge.Cuts) (width 0.15))
   (gr_line (start 93.98 133.985) (end 93.98 135.255) (angle 90) (layer Edge.Cuts) (width 0.15))
-  (gr_text 1.0 (at 144.145 127.635 90) (layer B.SilkS)
+  (gr_text 2.0 (at 144.145 127.635 90) (layer B.SilkS)
     (effects (font (size 5.08 3.81) (thickness 0.508)) (justify mirror))
   )
-  (gr_text "Sept 2017" (at 175.26 132.715) (layer F.SilkS)
+  (gr_text "Nov 2018" (at 175.26 132.715) (layer F.SilkS)
     (effects (font (size 1.5 1.5) (thickness 0.3)))
   )
